File: motor_driver/motor_driver.kicad_pcb (KiCad board)
At the start: 4 copper layers, 118 parts, among them J1 Conn_01x03_Pin, J2 Conn_01x05_Pin, J5 Conn_01x06_Pin, Q1 STB19NF20, Q2 STB19NF20, Q3 STB19NF20, Q4 STB19NF20, Q5 STB19NF20, Q6 STB19NF20, U1 AMC1302DWVR, U10 IR2110, U11 TLV6001DCK, U12 AMC1302DWVR, U13 TLV6001DCK, U15 IR2110, U16 TLV6001DCK, U3 IR2110, U4 TLV6001DCK, U5 TLV6001DCK, U6 uA7805, U7 AMC1302DWVR, U8 TLV6001DCK

Commit message: Minor component changes
Parts:
- added C40: 100nF, Capacitor_SMD:C_0603_1608Metric_Pad1.08x0.95mm_HandSolder, F.Cu at (268.8, 52.7)
- added C41: 22uF, Capacitor_SMD:C_0805_2012Metric_Pad1.18x1.45mm_HandSolder, F.Cu at (242.9, 58.9)
- added C42: 100nF, Capacitor_SMD:C_0603_1608Metric_Pad1.08x0.95mm_HandSolder, F.Cu at (268.8, 55.2)
- added C43: 22uF, Capacitor_SMD:C_0805_2012Metric_Pad1.18x1.45mm_HandSolder, F.Cu at (242.9, 61.9)
- added C44: 10nF, Capacitor_SMD:C_0402_1005Metric_Pad0.74x0.62mm_HandSolder, F.Cu at (203.8, 83.9)
- added C45: 100nF, Capacitor_SMD:C_0603_1608Metric_Pad1.08x0.95mm_HandSolder, F.Cu at (268.8, 57.7)
- added C46: 1uF, Capacitor_SMD:C_0805_2012Metric_Pad1.18x1.45mm_HandSolder, F.Cu at (242.9, 65.0)
- added C47: 100nF, Capacitor_SMD:C_0603_1608Metric_Pad1.08x0.95mm_HandSolder, F.Cu at (268.8, 60.2)
- added C48: 22uF, Capacitor_SMD:C_0805_2012Metric_Pad1.18x1.45mm_HandSolder, F.Cu at (242.9, 68.0)
- added C49: 330pF, Capacitor_SMD:C_0402_1005Metric_Pad0.74x0.62mm_HandSolder, F.Cu at (203.8, 85.8)
- added C50: 100nF, Capacitor_SMD:C_0603_1608Metric_Pad1.08x0.95mm_HandSolder, F.Cu at (268.8, 62.7)
- added C51: 22uF, Capacitor_SMD:C_0805_2012Metric_Pad1.18x1.45mm_HandSolder, F.Cu at (242.9, 71.0)
- added J3: Conn_01x03_Pin, Connector_PinHeader_2.54mm:PinHeader_1x03_P2.54mm_Vertical, F.Cu at (265.5, 74.0)
- added J4: Conn_01x06_Pin, Connector_PinHeader_2.54mm:PinHeader_1x06_P2.54mm_Vertical, F.Cu at (207.7, 71.4)
- C10, C27: value 100nF -> 10nF; footprint Capacitor_SMD:C_0603_1608Metric_Pad1.08x0.95mm_HandSolder -> Capacitor_SMD:C_0402_1005Metric_Pad0.74x0.62mm_HandSolder
- C11, C25, C30: value 330pF -> 100nF; footprint Capacitor_SMD:C_0402_1005Metric_Pad0.74x0.62mm_HandSolder -> Capacitor_SMD:C_0603_1608Metric_Pad1.08x0.95mm_HandSolder
- C12: value 330pF -> 1uF; footprint Capacitor_SMD:C_0402_1005Metric_Pad0.74x0.62mm_HandSolder -> Capacitor_SMD:C_0805_2012Metric_Pad1.18x1.45mm_HandSolder
- C14, C26, C31: value 100nF -> 22uF; footprint Capacitor_SMD:C_0603_1608Metric_Pad1.08x0.95mm_HandSolder -> Capacitor_SMD:C_0805_2012Metric_Pad1.18x1.45mm_HandSolder
- C15, C32: value 22uF -> 330pF; footprint Capacitor_SMD:C_0805_2012Metric -> Capacitor_SMD:C_0402_1005Metric_Pad0.74x0.62mm_HandSolder
- C17, C38: value 330pF -> 22uF; footprint Capacitor_SMD:C_0402_1005Metric_Pad0.74x0.62mm_HandSolder -> Capacitor_SMD:C_0805_2012Metric_Pad1.18x1.45mm_HandSolder
- C19, C2: value 22uF -> 1uF; footprint Capacitor_SMD:C_0805_2012Metric -> Capacitor_SMD:C_0805_2012Metric_Pad1.18x1.45mm_HandSolder
- C21, C24, C34, C4, C7, C9: footprint Capacitor_SMD:C_0805_2012Metric -> Capacitor_SMD:C_0805_2012Metric_Pad1.18x1.45mm_HandSolder
- C22, C5: value 10nF -> 330pF
- C28, C37: value 22uF -> 100nF; footprint Capacitor_SMD:C_0805_2012Metric -> Capacitor_SMD:C_0603_1608Metric_Pad1.08x0.95mm_HandSolder
- C29, C36: value 100nF -> 1uF; footprint Capacitor_SMD:C_0603_1608Metric_Pad1.08x0.95mm_HandSolder -> Capacitor_SMD:C_0805_2012Metric_Pad1.18x1.45mm_HandSolder
- C35: value 10nF -> 100nF; footprint Capacitor_SMD:C_0402_1005Metric_Pad0.74x0.62mm_HandSolder -> Capacitor_SMD:C_0603_1608Metric_Pad1.08x0.95mm_HandSolder
- C39: value 100nF -> 330pF; footprint Capacitor_SMD:C_0603_1608Metric_Pad1.08x0.95mm_HandSolder -> Capacitor_SMD:C_0402_1005Metric_Pad0.74x0.62mm_HandSolder
- D1, D3, D5: value 1N4007 -> UF4007
- J1: value Conn_01x03_Pin -> Conn_01x02_Pin; footprint Connector_PinHeader_2.54mm:PinHeader_1x03_P2.54mm_Vertical -> TerminalBlock:TerminalBlock_MaiXu_MX126-5.0-02P_1x02_P5.00mm
- J2: value Conn_01x05_Pin -> Conn_01x02_Pin; footprint Connector_PinHeader_1.00mm:PinHeader_1x05_P1.00mm_Vertical -> TerminalBlock:TerminalBlock_MaiXu_MX126-5.0-02P_1x02_P5.00mm
- J5: value Conn_01x06_Pin -> Conn_01x05_Pin; footprint Connector_PinHeader_2.54mm:PinHeader_1x06_P2.54mm_Vertical -> Connector_PinHeader_2.54mm:PinHeader_1x05_P2.54mm_Vertical
- R1: value 1k -> 3.3k
- R10: value 2k -> 100; footprint Resistor_SMD:R_1206_3216Metric -> Resistor_SMD:R_0805_2012Metric_Pad1.20x1.40mm_HandSolder
- R12: value 3.3k -> R_Shunt; footprint Resistor_SMD:R_0805_2012Metric_Pad1.20x1.40mm_HandSolder -> Custom_footprints:BVT-I-R003
- R13: value 3.3k -> 100
- R14: value 3.3k -> 10; footprint Resistor_SMD:R_0805_2012Metric_Pad1.20x1.40mm_HandSolder -> Resistor_SMD:R_1206_3216Metric_Pad1.30x1.75mm_HandSolder
- R2: value 1k -> 10; footprint Resistor_SMD:R_0805_2012Metric_Pad1.20x1.40mm_HandSolder -> Resistor_SMD:R_1206_3216Metric_Pad1.30x1.75mm_HandSolder
- R20, R36: value 2k -> 910; footprint Resistor_SMD:R_1206_3216Metric -> Resistor_SMD:R_1206_3216Metric_Pad1.30x1.75mm_HandSolder
- R3: value 30 -> 3.3k; footprint Resistor_SMD:R_1206_3216Metric_Pad1.30x1.75mm_HandSolder -> Resistor_SMD:R_0805_2012Metric_Pad1.20x1.40mm_HandSolder
- R4: value 100 -> 910; footprint Resistor_SMD:R_0805_2012Metric_Pad1.20x1.40mm_HandSolder -> Resistor_SMD:R_1206_3216Metric_Pad1.30x1.75mm_HandSolder
- R5: value R_Shunt -> 10; footprint Custom_footprints:BVT-I-R003 -> Resistor_SMD:R_1206_3216Metric_Pad1.30x1.75mm_HandSolder
- R6: value 100 -> 3.3k
- R7, R8: value 10 -> 1k; footprint Resistor_SMD:R_1206_3216Metric_Pad1.30x1.75mm_HandSolder -> Resistor_SMD:R_0805_2012Metric_Pad1.20x1.40mm_HandSolder
- R9: value 10 -> 30
- U1: value AMC1302DWVR -> uA7805; footprint Package_SO:SOIC-8_7.5x5.85mm_P1.27mm -> Package_TO_SOT_THT:TO-220-3_Vertical
- U11, U13, U16, U8: value TLV6001DCK -> TLV6001IDBVR; footprint Package_TO_SOT_SMD:SOT-353_SC-70-5 -> Package_TO_SOT_SMD:SOT-23-5_HandSoldering
- U2: value ~ -> AMC1302DWVR; footprint Custom_footprints:MCT6 -> Package_SO:SOIC-8_7.5x5.85mm_P1.27mm
- U3: value IR2110 -> TLV6001IDBVR; footprint Package_DIP:DIP-14_W7.62mm -> Package_TO_SOT_SMD:SOT-23-5_HandSoldering
- U4: value TLV6001DCK -> ~; footprint Package_TO_SOT_SMD:SOT-353_SC-70-5 -> Custom_footprints:MCT6
- U5: value TLV6001DCK -> IR2110; footprint Package_TO_SOT_SMD:SOT-353_SC-70-5 -> Package_DIP:DIP-14_W7.62mm
- U6: value uA7805 -> TLV6001IDBVR; footprint Package_TO_SOT_THT:TO-220-3_Vertical -> Package_TO_SOT_SMD:SOT-23-5_HandSoldering
- moved U6 71.3 mm to (190.2, 58.6)
- moved C28 68.2 mm to (264.4, 60.2)
- moved C37 68.1 mm to (264.4, 70.2)
- moved U5 66.6 mm to (145.1, 53.5)
- moved R10 65.1 mm to (195.5, 67.6)
- moved R14 63.7 mm to (248.3, 86.4)
- moved R4 63.0 mm to (248.3, 76.6)
- moved R2 62.9 mm to (248.3, 73.3)
- moved D2 55.7 mm to (145.6, 72.3)
- moved D4 55.7 mm to (145.6, 75.2)
- moved D6 55.7 mm to (145.6, 78.2)
- moved C19 49.8 mm to (238.1, 52.9)
- moved C21 49.8 mm to (238.1, 55.9)
- moved C24 49.8 mm to (238.1, 58.9)
- moved U2 48.8 mm to (223.9, 55.1)
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Connections:
- C1 pad 1: +5V -> +3.3V
- C1 pad 2: GND -> MCU_GND
- C10 pad 1: +3.3V -> Net-(C10-Pad1)
- C10 pad 2: MCU_GND -> Net-(C10-Pad2)
- C11 pad 1: Net-(U4--) -> Net-(D2-K)
- C11 pad 2: Net-(U5--) -> Net-(D2-A)
- C12 pad 1: /I_A -> Net-(D2-K)
- C12 pad 2: Net-(U4-+) -> Net-(D2-A)
- C13 pad 1: +3.3V -> Net-(D1-K)
- C13 pad 2: MCU_GND -> Net-(D2-A)
- C14 pad 1: +3.3V -> Net-(D1-K)
- C14 pad 2: MCU_GND -> Net-(D2-A)
- C15 pad 1: +3.3V -> Net-(U3--)
- C15 pad 2: MCU_GND -> Net-(U6--)
- C17 pad 1: /I_B -> +3.3V
- C17 pad 2: Net-(U8-+) -> MCU_GND
- C18 pad 1: +5V -> +3.3V
- C18 pad 2: GND -> MCU_GND
- C19 pad 1: +5V -> +3.3V
- C19 pad 2: GND -> MCU_GND
- C2 pad 1: +5V -> +3.3V
- C2 pad 2: GND -> MCU_GND
- C20 pad 1: +15V -> +3.3V
- C20 pad 2: GND -> MCU_GND
- C21 pad 1: +15V -> +3.3V
- C21 pad 2: GND -> MCU_GND
- C22 pad 1: Net-(C22-Pad1) -> /I_B
- C22 pad 2: Net-(C22-Pad2) -> Net-(U8-+)
- C23 pad 1: Net-(D3-K) -> +5V
- C23 pad 2: Net-(D4-A) -> GND
- C24 pad 1: Net-(D3-K) -> +5V
- C24 pad 2: Net-(D4-A) -> GND
- C25 pad 1: Net-(U8--) -> +15V
- C25 pad 2: Net-(U11--) -> GND
- C26 pad 1: +3.3V -> +15V
- C26 pad 2: MCU_GND -> GND
- C27 pad 1: +3.3V -> Net-(C27-Pad1)
- C27 pad 2: MCU_GND -> Net-(C27-Pad2)
- C28 pad 1: +3.3V -> Net-(D4-K)
- C28 pad 2: MCU_GND -> Net-(D4-A)
- C29 pad 1: +3.3V -> Net-(D4-K)
- C29 pad 2: MCU_GND -> Net-(D4-A)
- C3 pad 1: +15V -> +3.3V
- C3 pad 2: GND -> MCU_GND
- C30 pad 1: /I_C -> Net-(D3-K)
- C30 pad 2: Net-(U13-+) -> Net-(D4-A)
- C31 pad 1: +5V -> Net-(D3-K)
- C31 pad 2: GND -> Net-(D4-A)
- C32 pad 1: +5V -> Net-(U8--)
- C32 pad 2: GND -> Net-(U11--)
- C33 pad 1: +15V -> +3.3V
- C33 pad 2: GND -> MCU_GND
- C34 pad 1: +15V -> +3.3V
- C34 pad 2: GND -> MCU_GND
- C35 pad 1: Net-(C35-Pad1) -> +3.3V
- C35 pad 2: Net-(C35-Pad2) -> MCU_GND
- C36 pad 1: Net-(D5-K) -> +3.3V
- C36 pad 2: Net-(D6-A) -> MCU_GND
- C37 pad 1: Net-(D5-K) -> +3.3V
- C37 pad 2: Net-(D6-A) -> MCU_GND
- C38 pad 1: Net-(U13--) -> +3.3V
- C38 pad 2: Net-(U16--) -> MCU_GND
- C39 pad 1: +3.3V -> /I_C
- C39 pad 2: MCU_GND -> Net-(U13-+)
- C4 pad 1: +15V -> +3.3V
- C4 pad 2: GND -> MCU_GND
- C5 pad 1: Net-(C5-Pad1) -> /I_A
- C5 pad 2: Net-(C5-Pad2) -> Net-(U3-+)
- C6 pad 1: Net-(D1-K) -> +5V
- C6 pad 2: Net-(D2-A) -> GND
- C7 pad 1: Net-(D1-K) -> +5V
- C7 pad 2: Net-(D2-A) -> GND
- C8 pad 1: +3.3V -> +15V
- C8 pad 2: MCU_GND -> GND
- C9 pad 1: +3.3V -> +15V
- C9 pad 2: MCU_GND -> GND
- J1 pad 1: /PHASE_A -> +100V
- J1 pad 2: /PHASE_B -> GND
- J2 pad 1: /I_A -> +15V
- J2 pad 2: /I_B -> GND
- J5 pad 1: /HI_A -> /I_A
- J5 pad 2: /LO_A -> /I_B
- J5 pad 3: /HI_B -> /I_C
- J5 pad 4: /LO_B -> +3.3V
- J5 pad 5: /HI_C -> MCU_GND
- R1 pad 1: +5V -> Net-(U3-+)
- R1 pad 2: Net-(U3-HIN) -> /I_A
- R10 pad 1: Net-(D2-K) -> /HI_A
- R10 pad 2: Net-(D1-K) -> Net-(R10-Pad2)
- R11 pad 1: Net-(U1-OUTN) -> Net-(U3--)
- R11 pad 2: Net-(U4--) -> Net-(U6--)
- R12 pad 1: Net-(U1-OUTP) -> Net-(D2-A)
- R12 pad 2: Net-(U4-+) -> Net-(C10-Pad2)
- R13 pad 1: Net-(U4-+) -> /LO_A
- R13 pad 2: /I_A -> Net-(R13-Pad2)
- R14 pad 1: Net-(U4--) -> Net-(U5-LO)
- R14 pad 2: Net-(U5--) -> Net-(Q2-G)
- R15 pad 2: Net-(U5-+) -> Net-(U6-+)
- R16 pad 1: Net-(U5-+) -> Net-(U6-+)
- R18 pad 1: Net-(C22-Pad1) -> Net-(C27-Pad1)
- R2 pad 1: +5V -> Net-(C10-Pad1)
- R2 pad 2: Net-(U3-LIN) -> Net-(U2-INP)
- R21 pad 1: Net-(C22-Pad2) -> Net-(C27-Pad2)
- R28 pad 2: Net-(C22-Pad2) -> Net-(C27-Pad2)
- R28 pad 3: Net-(C22-Pad1) -> Net-(C27-Pad1)
- R3 pad 1: Net-(U3-HO) -> Net-(U2-OUTP)
- R3 pad 2: Net-(Q1-G) -> Net-(U3-+)
- R34 pad 1: Net-(C35-Pad1) -> Net-(C44-Pad1)
- R37 pad 1: Net-(C35-Pad2) -> Net-(C44-Pad2)
- R4 pad 1: /HI_A -> Net-(D2-K)
- R4 pad 2: Net-(R4-Pad2) -> Net-(D1-K)
- R44 pad 2: Net-(C35-Pad2) -> Net-(C44-Pad2)
- R44 pad 3: Net-(C35-Pad1) -> Net-(C44-Pad1)
- R5 pad 1: Net-(D2-A) -> Net-(C10-Pad2)
- R5 pad 2: Net-(C5-Pad2) -> Net-(U2-INN)
- R6 pad 1: /LO_A -> Net-(U2-OUTN)
- R6 pad 2: Net-(R6-Pad2) -> Net-(U3--)
- R7 pad 1: Net-(U3-LO) -> +5V
- R7 pad 2: Net-(Q2-G) -> Net-(U5-HIN)
- R8 pad 1: Net-(C5-Pad1) -> +5V
- R8 pad 2: Net-(U1-INP) -> Net-(U5-LIN)
- R9 pad 1: Net-(C5-Pad2) -> Net-(U5-HO)
- R9 pad 2: Net-(U1-INN) -> Net-(Q1-G)
- U1 pad 1: Net-(D2-K) -> +15V
- U1 pad 2: Net-(U1-INP) -> GND
- U1 pad 3: Net-(U1-INN) -> +5V
- U2 pad 1: Net-(R4-Pad2) -> Net-(D2-K)
- U2 pad 2: MCU_GND -> Net-(U2-INP)
- U2 pad 3: MCU_GND -> Net-(U2-INN)
- U2 pad 4: Net-(R6-Pad2) -> Net-(D2-A)
- U2 pad 5: GND -> MCU_GND
- U2 pad 6: Net-(U3-LIN) -> Net-(U2-OUTN)
- U2 pad 7: Net-(U3-HIN) -> Net-(U2-OUTP)
- U2 pad 8: GND -> +3.3V
- U3 pad 1: Net-(U3-LO) -> Net-(U3-+)
- U3 pad 2: GND -> MCU_GND
- U3 pad 3: +15V -> Net-(U3--)
- U3 pad 4: unconnected-(U3-NC-Pad4) -> /I_A
- U3 pad 5: Net-(D2-A) -> +3.3V
- U4 pad 1: Net-(U4-+) -> Net-(R10-Pad2)
- U4 pad 3: Net-(U4--) -> MCU_GND
- U4 pad 4: /I_A -> Net-(R13-Pad2)
- U4 pad 5: +3.3V -> GND
- U5 pad 1: Net-(U5-+) -> Net-(U5-LO)
- U5 pad 2: MCU_GND -> GND
- U5 pad 3: Net-(U5--) -> +15V
- U5 pad 4: Net-(U5--) -> unconnected-(U5-NC-Pad4)
- U5 pad 5: +3.3V -> Net-(D2-A)
- U6 pad 1: +15V -> Net-(U6-+)
- U6 pad 2: GND -> MCU_GND
- U6 pad 3: +5V -> Net-(U6--)

Commit message: WIP
Parts:
- removed D4, D6: BZX384xxxx, Diode_SMD:D_SOD-323
- removed D5: UF4007, Diode_THT:D_DO-41_SOD81_P10.16mm_Horizontal
- added C52: 100nF, Capacitor_SMD:C_0603_1608Metric_Pad1.08x0.95mm_HandSolder, F.Cu at (43.1, 102.2)
- added C53: 330nF, Capacitor_SMD:C_0805_2012Metric_Pad1.18x1.45mm_HandSolder, F.Cu at (36.0, 102.0)
- added U17: LM4040DBZ-5, Package_TO_SOT_SMD:SOT-23, F.Cu at (141.8, 67.9)
- added U18: IR2110, Package_DIP:DIP-14_W7.62mm, F.Cu at (58.2, 110.0)
- added U19: TLV6001IDBVR, Package_TO_SOT_SMD:SOT-23-5_HandSoldering, B.Cu at (210.5, 43.5)
- C1, C15, C16, C17, C18, C19, C2, C20, C21, C22, C3, C32, C33, C34, C35, C36, C37, C38, C39, C4, C49, C5, C50, C51, R1, R11, R15, R16, R17, R19, R22, R27, R3, R31, R32, R33, R35, R38, R43, R47, R48, R6, U3, U6, U8: moved to B.Cu
- D2: value BZX384xxxx -> UF4007; footprint Diode_SMD:D_SOD-323 -> Diode_THT:D_DO-41_SOD81_P10.16mm_Horizontal
- J1: footprint TerminalBlock:TerminalBlock_MaiXu_MX126-5.0-02P_1x02_P5.00mm -> TerminalBlock_MetzConnect:TerminalBlock_MetzConnect_Type067_RT01902HDWC_1x02_P10.00mm_Horizontal
- J3: footprint Connector_PinHeader_2.54mm:PinHeader_1x03_P2.54mm_Vertical -> TerminalBlock_MetzConnect:TerminalBlock_MetzConnect_Type067_RT01903HDWC_1x03_P10.00mm_Horizontal
- Q1, Q2, Q3, Q4, Q5, Q6: footprint Custom_footprints:STB19NF20 -> Custom_footprints:TO-220-3_Vertical_Heat_Sink
- R20, R36, R4: value 910 -> 1k
- R28: footprint Custom_footprints:BVT-I-R003 -> Custom_footprints:BVT-I-R003_Reverse
- U10: value IR2110 -> LM4040DBZ-5; footprint Package_DIP:DIP-14_W7.62mm -> Package_TO_SOT_SMD:SOT-23
- U11: value TLV6001IDBVR -> IR2110; footprint Package_TO_SOT_SMD:SOT-23-5_HandSoldering -> Package_DIP:DIP-14_W7.62mm
- U12: value AMC1302DWVR -> TLV6001IDBVR; footprint Package_SO:SOIC-8_7.5x5.85mm_P1.27mm -> Package_TO_SOT_SMD:SOT-23-5_HandSoldering; moved to B.Cu
- U13: value TLV6001IDBVR -> AMC1302DWVR; footprint Package_TO_SOT_SMD:SOT-23-5_HandSoldering -> Package_SO:SOIC-8_7.5x5.85mm_P1.27mm
- U14: value ~ -> TLV6001IDBVR; footprint Custom_footprints:MCT6 -> Package_TO_SOT_SMD:SOT-23-5_HandSoldering; moved to B.Cu
- U15: value IR2110 -> ~; footprint Package_DIP:DIP-14_W7.62mm -> Custom_footprints:MCT6
- U16: value TLV6001IDBVR -> LM4040DBZ-5; footprint Package_TO_SOT_SMD:SOT-23-5_HandSoldering -> Package_TO_SOT_SMD:SOT-23
- moved C40 225.4 mm to (47.6, 96.5), turned to 180 degrees
- moved C23 218.0 mm to (47.6, 78.5), turned to 180 degrees
- moved C42 213.0 mm to (61.4, 104.0)
- moved C6 212.4 mm to (47.6, 58.8), turned to 180 degrees
- moved C47 211.8 mm to (60.5, 98.9), turned to -90 degrees
- moved J2 209.8 mm to (46.2, 119.0)
- moved C25 204.8 mm to (61.4, 84.8)
- moved C30 204.6 mm to (60.5, 79.6), turned to -90 degrees
- moved C13 199.6 mm to (60.5, 60.1), turned to -90 degrees
- moved C8 198.7 mm to (61.4, 65.0)
- moved C41 198.7 mm to (47.5, 94.5), turned to 180 degrees
- moved R46 195.9 mm to (66.0, 111.5)
- moved R41 194.6 mm to (66.0, 95.2)
- moved C24 191.5 mm to (47.5, 76.5), turned to 180 degrees
- moved J1 191.1 mm to (68.8, 119.0), turned to 180 degrees
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Connections:
- C10 pad 1: Net-(C10-Pad1) -> Net-(U2-INP)
- C10 pad 2: Net-(C10-Pad2) -> Net-(U2-INN)
- C11 pad 1: Net-(D2-K) -> Net-(U17-K)
- C11 pad 2: Net-(D2-A) -> Net-(Q1-S)
- C12 pad 1: Net-(D2-K) -> Net-(U17-K)
- C12 pad 2: Net-(D2-A) -> Net-(Q1-S)
- C13 pad 2: Net-(D2-A) -> Net-(Q1-S)
- C14 pad 2: Net-(D2-A) -> Net-(Q1-S)
- C27 pad 1: Net-(C27-Pad1) -> Net-(U7-INP)
- C27 pad 2: Net-(C27-Pad2) -> Net-(U7-INN)
- C28 pad 1: Net-(D4-K) -> Net-(U10-K)
- C28 pad 2: Net-(D4-A) -> Net-(Q3-S)
- C29 pad 1: Net-(D4-K) -> Net-(U10-K)
- C29 pad 2: Net-(D4-A) -> Net-(Q3-S)
- C30 pad 1: Net-(D3-K) -> Net-(D2-K)
- C30 pad 2: Net-(D4-A) -> Net-(Q3-S)
- C31 pad 1: Net-(D3-K) -> Net-(D2-K)
- C31 pad 2: Net-(D4-A) -> Net-(Q3-S)
- C32 pad 2: Net-(U11--) -> Net-(U12--)
- C39 pad 2: Net-(U13-+) -> Net-(U14-+)
- C44 pad 1: Net-(C44-Pad1) -> Net-(U13-INP)
- C44 pad 2: Net-(C44-Pad2) -> Net-(U13-INN)
- C45 pad 1: Net-(D6-K) -> Net-(U13-VDD1)
- C45 pad 2: Net-(D6-A) -> Net-(Q5-S)
- C46 pad 1: Net-(D6-K) -> Net-(U13-VDD1)
- C46 pad 2: Net-(D6-A) -> Net-(Q5-S)
- C47 pad 1: Net-(D5-K) -> Net-(D3-K)
- C47 pad 2: Net-(D6-A) -> Net-(Q5-S)
- C48 pad 1: Net-(D5-K) -> Net-(D3-K)
- C48 pad 2: Net-(D6-A) -> Net-(Q5-S)
- C49 pad 1: Net-(U13--) -> Net-(U14--)
- C49 pad 2: Net-(U16--) -> Net-(U19--)
- D2 pad 2: Net-(D2-A) -> +15V
- Q1 pad 3: Net-(D2-A) -> Net-(Q1-S)
- Q2 pad 2: Net-(D2-A) -> Net-(Q1-S)
- Q3 pad 3: Net-(D4-A) -> Net-(Q3-S)
- Q4 pad 2: Net-(D4-A) -> Net-(Q3-S)
- Q5 pad 3: Net-(D6-A) -> Net-(Q5-S)
- Q6 pad 2: Net-(D6-A) -> Net-(Q5-S)
- R12 pad 1: Net-(D2-A) -> Net-(Q1-S)
- R12 pad 2: Net-(C10-Pad2) -> Net-(R12-Pad2)
- R12 pad 3: Net-(C10-Pad1) -> Net-(R12-Pad3)
- R18 pad 1: Net-(C27-Pad1) -> Net-(R18-Pad1)
- R2 pad 1: Net-(C10-Pad1) -> Net-(R12-Pad3)
- R20 pad 1: Net-(D4-K) -> Net-(U10-K)
- R20 pad 2: Net-(D3-K) -> Net-(D2-K)
- R21 pad 1: Net-(C27-Pad2) -> Net-(R21-Pad1)
- R23 pad 2: Net-(U10-HIN) -> Net-(U11-HIN)
- R24 pad 2: Net-(U10-LIN) -> Net-(U11-LIN)
- R25 pad 1: Net-(U10-HO) -> Net-(U11-HO)
- R27 pad 2: Net-(U11--) -> Net-(U12--)
- R28 pad 1: Net-(D4-A) -> Net-(Q3-S)
- R28 pad 2: Net-(C27-Pad2) -> Net-(R21-Pad1)
- R28 pad 3: Net-(C27-Pad1) -> Net-(R18-Pad1)
- R30 pad 1: Net-(U10-LO) -> Net-(U11-LO)
- R31 pad 2: Net-(U11-+) -> Net-(U12-+)
- R32 pad 1: Net-(U11-+) -> Net-(U12-+)
- R33 pad 1: Net-(U13-+) -> Net-(U14-+)
- R34 pad 1: Net-(C44-Pad1) -> Net-(R34-Pad1)
- R34 pad 2: Net-(U12-INP) -> Net-(U13-INP)
- R35 pad 1: Net-(U12-OUTP) -> Net-(U13-OUTP)
- R35 pad 2: Net-(U13-+) -> Net-(U14-+)
- R36 pad 1: Net-(D6-K) -> Net-(U13-VDD1)
- R36 pad 2: Net-(D5-K) -> Net-(D3-K)
- R37 pad 1: Net-(C44-Pad2) -> Net-(R37-Pad1)
- R37 pad 2: Net-(U12-INN) -> Net-(U13-INN)
- R38 pad 1: Net-(U12-OUTN) -> Net-(U13-OUTN)
- R38 pad 2: Net-(U13--) -> Net-(U14--)
- R39 pad 2: Net-(U15-HIN) -> Net-(U18-HIN)
- R4 pad 1: Net-(D2-K) -> Net-(U17-K)
- R40 pad 2: Net-(U15-LIN) -> Net-(U18-LIN)
- R41 pad 1: Net-(U15-HO) -> Net-(U18-HO)
- R43 pad 1: Net-(U13--) -> Net-(U14--)
- R43 pad 2: Net-(U16--) -> Net-(U19--)
- R44 pad 1: Net-(D6-A) -> Net-(Q5-S)
- R44 pad 2: Net-(C44-Pad2) -> Net-(R37-Pad1)
- R44 pad 3: Net-(C44-Pad1) -> Net-(R34-Pad1)
- R46 pad 1: Net-(U15-LO) -> Net-(U18-LO)
- R47 pad 2: Net-(U16-+) -> Net-(U19-+)
- R48 pad 1: Net-(U16-+) -> Net-(U19-+)
- R5 pad 1: Net-(C10-Pad2) -> Net-(R12-Pad2)
- U10 pad 1: Net-(U10-LO) -> Net-(U10-K)
- U10 pad 2: GND -> Net-(Q3-S)
- U10 pad 3: +15V -> unconnected-(U10-NC-Pad3)
- U11 pad 1: Net-(U11-+) -> Net-(U11-LO)
- U11 pad 2: MCU_GND -> GND
- U11 pad 3: Net-(U11--) -> +15V
- U11 pad 4: Net-(U11--) -> unconnected-(U11-NC-Pad4)
- U11 pad 5: +3.3V -> Net-(Q3-S)
- U12 pad 1: Net-(D6-K) -> Net-(U12-+)
- U12 pad 2: Net-(U12-INP) -> MCU_GND
- U12 pad 3: Net-(U12-INN) -> Net-(U12--)
- U12 pad 4: Net-(D6-A) -> Net-(U12--)
- U12 pad 5: MCU_GND -> +3.3V
- U13 pad 1: Net-(U13-+) -> Net-(U13-VDD1)
- U13 pad 2: MCU_GND -> Net-(U13-INP)
- U13 pad 3: Net-(U13--) -> Net-(U13-INN)
- U13 pad 4: /I_C -> Net-(Q5-S)
- U13 pad 5: +3.3V -> MCU_GND
- U14 pad 1: Net-(R42-Pad2) -> Net-(U14-+)
- U14 pad 3: MCU_GND -> Net-(U14--)
- U14 pad 4: Net-(R45-Pad2) -> /I_C
- U14 pad 5: GND -> +3.3V
- U15 pad 1: Net-(U15-LO) -> Net-(R42-Pad2)
- U15 pad 2: GND -> MCU_GND
- U15 pad 3: +15V -> MCU_GND
- U15 pad 4: unconnected-(U15-NC-Pad4) -> Net-(R45-Pad2)
- U15 pad 5: Net-(D6-A) -> GND
- U15 pad 6: Net-(D5-K) -> Net-(U18-LIN)
- U15 pad 7: Net-(U15-HO) -> Net-(U18-HIN)
- U15 pad 8: unconnected-(U15-NC-Pad8) -> GND
- U16 pad 1: Net-(U16-+) -> Net-(U13-VDD1)
- U16 pad 2: MCU_GND -> Net-(Q5-S)
- U16 pad 3: Net-(U16--) -> unconnected-(U16-NC-Pad3)
- U2 pad 1: Net-(D2-K) -> Net-(U17-K)
- U2 pad 4: Net-(D2-A) -> Net-(Q1-S)
- U5 pad 5: Net-(D2-A) -> Net-(Q1-S)
- U7 pad 1: Net-(D4-K) -> Net-(U10-K)
- U7 pad 4: Net-(D4-A) -> Net-(Q3-S)
- U9 pad 6: Net-(U10-LIN) -> Net-(U11-LIN)
- U9 pad 7: Net-(U10-HIN) -> Net-(U11-HIN)
Routing:
- net Net-(D3-K): track 0.00 -> 103.2 mm, vias 0 -> 1
- net Net-(D2-K): track 0.00 -> 91.0 mm, vias 0 -> 1
- net Net-(Q5-S): track 0.00 -> 80.9 mm, vias 0 -> 12
- net Net-(D1-K): track 0.00 -> 79.3 mm, vias 0 -> 1
- net Net-(Q4-G): track 0.00 -> 61.7 mm
- net Net-(Q2-G): track 0.00 -> 50.8 mm
- net Net-(Q6-G): track 0.00 -> 50.2 mm
- net Net-(Q3-S): track 0.00 -> 39.8 mm, vias 0 -> 8
- net +15V: track 0.00 -> 37.5 mm
- net GND: track 0.00 -> 36.9 mm, vias 0 -> 15
- net +5V: track 0.00 -> 29.4 mm, vias 0 -> 6
- net Net-(Q3-G): track 0.00 -> 27.9 mm
- net Net-(Q1-S): track 0.00 -> 26.2 mm, vias 0 -> 8
- net Net-(Q5-G): track 0.00 -> 23.8 mm
- net Net-(Q1-G): track 0.00 -> 16.4 mm
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- added copper zone on In1.Cu, net +100V
- added copper zone on In1.Cu, net +15V
- added copper zone on In1.Cu, net +5V
- added copper zone on F.Cu, net /PHASE_A
- added copper zone on In1.Cu, net /PHASE_A
- added copper zone on F.Cu, net /PHASE_B
- added copper zone on In1.Cu, net /PHASE_B
- added copper zone on F.Cu, net /PHASE_C
- added copper zone on In1.Cu, net /PHASE_C
- added copper zone on In2.Cu, net GND
- added copper zone on In1.Cu, net MCU_GND
- added copper zone on F.Cu, net Net-(Q1-S)
- added copper zone on In1.Cu, net Net-(Q1-S)
- added copper zone on F.Cu, net Net-(Q3-S)
- added copper zone on In1.Cu, net Net-(Q3-S)
- added copper zone on F.Cu, net Net-(Q5-S)
- added copper zone on In1.Cu, net Net-(Q5-S)

Commit message: Almost done
Parts:
- C1, C15, C16, C17, C18, C19, C2, C20, C21, C22, C3, C32, C33, C34, C35, C36, C37, C38, C39, C4, C49, C5, C50, C51, R1, R11, R15, R16, R17, R19, R22, R27, R3, R31, R32, R33, R35, R38, R43, R47, R48, R6, U12, U14, U19, U3, U6, U8: moved to F.Cu
- moved U19 131.1 mm to (80.6, 61.5), turned to -90 degrees
- moved R1 130.4 mm to (92.0, 54.0)
- moved U14 128.6 mm to (86.0, 70.7), turned to -90 degrees
- moved R17 126.6 mm to (92.2, 44.9)
- moved C49 126.5 mm to (85.2, 65.6), turned to 90 degrees
- moved R6 126.4 mm to (96.0, 54.0)
- moved C3 126.1 mm to (89.1, 57.0)
- moved R33 126.0 mm to (83.0, 71.7), turned to -90 degrees
- moved C39 125.5 mm to (81.4, 71.6), turned to 90 degrees
- moved R38 125.4 mm to (82.8, 67.0), turned to -90 degrees
- moved C22 124.6 mm to (93.0, 46.5), turned to 0 degrees
- moved R3 124.5 mm to (98.0, 58.7)
- moved C20 124.0 mm to (89.3, 47.6)
- moved U3 123.1 mm to (93.5, 57.9)
- moved C32 122.8 mm to (97.5, 47.3), turned to 90 degrees
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Connections:
- C15 pad 1: Net-(U3--) -> Net-(U3-+)
- C22 pad 2: Net-(U8-+) -> Net-(U8--)
- C32 pad 1: Net-(U8--) -> Net-(U8-+)
- C39 pad 2: Net-(U14-+) -> Net-(U14--)
- C49 pad 1: Net-(U14--) -> Net-(U14-+)
- C5 pad 2: Net-(U3-+) -> Net-(U3--)
- J5 pad 4: +3.3V -> MCU_GND
- J5 pad 5: MCU_GND -> +3.3V
- R1 pad 1: Net-(U3-+) -> Net-(U3--)
- R11 pad 1: Net-(U3--) -> Net-(U3-+)
- R17 pad 1: Net-(U8-+) -> Net-(U8--)
- R27 pad 1: Net-(U8--) -> Net-(U8-+)
- R33 pad 1: Net-(U14-+) -> Net-(U14--)
- R43 pad 1: Net-(U14--) -> Net-(U14-+)
Routing:
- net MCU_GND: track 0.00 -> 286.7 mm, vias 0 -> 30
- net +3.3V: track 0.00 -> 278.9 mm, vias 0 -> 15
- net Net-(U13-OUTN): track 0.00 -> 197.2 mm, vias 0 -> 3
- net Net-(U13-OUTP): track 0.00 -> 191.2 mm, vias 0 -> 2
- net Net-(U7-OUTN): track 0.00 -> 165.6 mm, vias 0 -> 2
- net Net-(U7-OUTP): track 0.00 -> 163.8 mm, vias 0 -> 2
- net Net-(U2-OUTP): track 0.00 -> 116.5 mm, vias 0 -> 3
- net Net-(U2-OUTN): track 0.00 -> 111.6 mm, vias 0 -> 2
- net /I_B: track 0.00 -> 42.0 mm
- net /I_A: track 0.00 -> 33.9 mm
- net Net-(Q1-S): track 26.2 -> 54.2 mm, vias 8 -> 12
- net Net-(Q3-S): track 39.8 -> 67.0 mm, vias 8 -> 12
- net Net-(U10-K): track 0.00 -> 16.6 mm
- net Net-(U6--): track 0.00 -> 13.8 mm
- net Net-(U12--): track 0.00 -> 13.8 mm
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- added copper zone on In1.Cu, net +3.3V
- added copper zone on B.Cu, net MCU_GND

Commit message: Done
Connections:
- R12 pad 2: Net-(R12-Pad2) -> /PHASE_A
- R18 pad 1: Net-(R18-Pad1) -> /PHASE_B
- R2 pad 1: Net-(R12-Pad3) -> /PHASE_A
- R21 pad 1: Net-(R21-Pad1) -> Net-(Q3-S)
- R28 pad 2: Net-(R21-Pad1) -> /PHASE_B
- R34 pad 1: Net-(R34-Pad1) -> /PHASE_C
- R37 pad 1: Net-(R37-Pad1) -> Net-(Q5-S)
- R44 pad 2: Net-(R37-Pad1) -> /PHASE_C
- R5 pad 1: Net-(R12-Pad2) -> Net-(Q1-S)
Routing:
- net Net-(Q5-S): track 80.9 -> 94.9 mm
- net /PHASE_B: track 0.00 -> 11.0 mm
- net /PHASE_C: track 0.00 -> 10.8 mm
- net Net-(R37-Pad1): track 10.3 -> 0.00 mm
- net /PHASE_A: track 0.00 -> 9.93 mm
- net Net-(Q1-S): track 54.2 -> 61.9 mm
- net Net-(R34-Pad1): track 7.17 -> 0.00 mm
- net Net-(Q3-S): track 67.0 -> 74.2 mm
- net Net-(R18-Pad1): track 6.43 -> 0.00 mm
- net Net-(R12-Pad3): track 6.32 -> 0.00 mm
- net Net-(R12-Pad2): track 2.89 -> 0.00 mm
- net Net-(R21-Pad1): track 2.81 -> 0.00 mm
- net MCU_GND: track 286.7 -> 285.5 mm
- net GND: vias 15 -> 92
- net (no net): vias 0 -> 4
- added copper zone on F.Cu, net GND
- removed copper zone on F.Cu, net /PHASE_A
- removed copper zone on F.Cu, net /PHASE_B
- removed copper zone on F.Cu, net /PHASE_C
- removed copper zone on F.Cu, net Net-(Q1-S)
- removed copper zone on F.Cu, net Net-(Q3-S)
- removed copper zone on F.Cu, net Net-(Q5-S)
Other:
- board outline added: 144.5 x 107 mm
- board text added: "+100V"
- board text added: "+15V"
- board text added: "+3V3 GND IC IB IA"
- board text added: ":D"
- board text added: "A"
- board text added: "A'"
- board text added: "AMY LI FEB. 2025"
- board text added: "B"
- board text added: "B'"
- board text added: "C"
- board text added: "C B A"
- board text added: "C'"
- board text added: "C' C B' B A' A"
- board text added: "GND"
- board text added: "IAN"
- board text added: "IAP"
- board text added: "IBN"
- board text added: "IBP"
- board text added: "ICN"
- board text added: "ICP"
- board text added: "MINI MAGLEV DRIVER V1"
- board text added: "VDD1"

Commit message: Add 3d models
Parts:
- J1: footprint TerminalBlock_MetzConnect:TerminalBlock_MetzConnect_Type067_RT01902HDWC_1x02_P10.00mm_Horizontal -> Custom_footprints:TerminalBlock_MetzConnect_Type067_RT01902HDWC_1x02_P10.00mm_Horizontal
- J2: footprint TerminalBlock:TerminalBlock_MaiXu_MX126-5.0-02P_1x02_P5.00mm -> Custom_footprints:TerminalBlock_MaiXu_MX126-5.0-02P_1x02_P5.00mm
- J3: footprint TerminalBlock_MetzConnect:TerminalBlock_MetzConnect_Type067_RT01903HDWC_1x03_P10.00mm_Horizontal -> Custom_footprints:TerminalBlock_MetzConnect_Type067_RT01903HDWC_1x03_P10.00mm_Horizontal
- U13, U2, U7: footprint Package_SO:SOIC-8_7.5x5.85mm_P1.27mm -> Custom_footprints:SOIC-8_7.5x5.85mm_P1.27mm
- moved J2 2.57 mm to (94.5, 133.8)
- moved J1 2.14 mm to (117.5, 133.5)
- moved J3 1.50 mm to (208.0, 113.8)
Routing:
- net +15V: track 37.5 -> 39.2 mm
