File: motor_driver/motor_driver.kicad_pcb (KiCad board)
At the start: 4 copper layers, 144.5 x 107 mm, 134 parts, among them J1 Conn_01x02_Pin, J2 Conn_01x02_Pin, J3 Conn_01x03_Pin, J4 Conn_01x06_Pin, J5 Conn_01x05_Pin, Q1 STB19NF20, Q2 STB19NF20, Q3 STB19NF20, Q4 STB19NF20, Q5 STB19NF20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

Commit message: Minor formatting change
Other:
- board text added: "AMY L. FEB. 2025"
- board text removed: "AMY LI FEB. 2025"
Changed lines of the file:
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@@
 		(layer "Edge.Cuts")
 	)
-	(gr_text "AMY LI\nFEB. 2025"
+	(gr_text "AMY L.\nFEB. 2025"
 		(at 178.25 62.2 0)
 		(layer "F.SilkS")
