File: motor_driver/motor_driver.kicad_sch (KiCad schematic)
At the start: 132 parts, among them J1 Conn_01x02_Pin, J2 Conn_01x02_Pin, J3 Conn_01x03_Pin, J4 Conn_01x06_Pin, J5 Conn_01x05_Pin, Q1 STB19NF20, Q2 STB19NF20, Q3 STB19NF20, Q4 STB19NF20, Q5 STB19NF20, Q6 STB19NF20, U1 uA7805, U10 IR2110, U11 TLV6001IDBVR, U12 AMC1302DWVR, U13 TLV6001IDBVR, U15 IR2110, U16 TLV6001IDBVR, U2 AMC1302DWVR, U3 TLV6001IDBVR, U5 IR2110, U6 TLV6001IDBVR, U7 AMC1302DWVR, U8 TLV6001IDBVR

Commit message: WIP
Parts:
- removed D2, D4, D6: BZX384xxxx, Diode_SMD:D_SOD-323, symbol Diode:BZX384xxxx
- removed D5: UF4007, Diode_THT:D_DO-41_SOD81_P10.16mm_Horizontal, symbol Diode:1N4007
- removed U10, U15: IR2110, Package_DIP:DIP-14_W7.62mm, symbol Driver_FET:IR2110
- removed U11, U13, U16: TLV6001IDBVR, Package_TO_SOT_SMD:SOT-23-5_HandSoldering, symbol Amplifier_Operational:TLV6001DCK
- removed U12: AMC1302DWVR, Package_SO:SOIC-8_7.5x5.85mm_P1.27mm, symbol Custom_schematics:AMC1302DWVR
- removed U14: ~, Custom_footprints:MCT6, symbol Custom_schematics:MCT6
- added C52: 100nF, Capacitor_SMD:C_0603_1608Metric_Pad1.08x0.95mm_HandSolder, symbol Device:C
- added C53: 330nF, Capacitor_SMD:C_0805_2012Metric_Pad1.18x1.45mm_HandSolder, symbol Device:C
- added D2: UF4007, Diode_THT:D_DO-41_SOD81_P10.16mm_Horizontal, symbol Diode:1N4007
- added U10, U16, U17: LM4040DBZ-5, Package_TO_SOT_SMD:SOT-23, symbol Reference_Voltage:LM4040DBZ-5
- added U11, U18: IR2110, Package_DIP:DIP-14_W7.62mm, symbol Driver_FET:IR2110
- added U12, U14, U19: TLV6001IDBVR, Package_TO_SOT_SMD:SOT-23-5_HandSoldering, symbol Amplifier_Operational:TLV6001DCK
- added U13: AMC1302DWVR, Package_SO:SOIC-8_7.5x5.85mm_P1.27mm, symbol Custom_schematics:AMC1302DWVR
- added U15: ~, Custom_footprints:MCT6, symbol Custom_schematics:MCT6
- J1: footprint TerminalBlock:TerminalBlock_MaiXu_MX126-5.0-02P_1x02_P5.00mm -> TerminalBlock_MetzConnect:TerminalBlock_MetzConnect_Type067_RT01902HDWC_1x02_P10.00mm_Horizontal
- J3: footprint Connector_PinHeader_2.54mm:PinHeader_1x03_P2.54mm_Vertical -> TerminalBlock_MetzConnect:TerminalBlock_MetzConnect_Type067_RT01903HDWC_1x03_P10.00mm_Horizontal
- Q1, Q2, Q3, Q4, Q5, Q6: footprint Custom_footprints:STB19NF20 -> Custom_footprints:TO-220-3_Vertical_Heat_Sink
- R20, R36, R4: value 910 -> 1k
- R28: footprint Custom_footprints:BVT-I-R003 -> Custom_footprints:BVT-I-R003_Reverse
Connections:
- net +15V: now also C53.1, D2.2 (A), U11.3 (VCC), U18.3 (VCC)
- net +3.3V: now also U12.5 (V+), U13.8 (VDD2), U14.5 (V+), U19.5 (V+)
- net +5V: now also C52.1, U11.9 (VDD), U18.9 (VDD)
- net GND: now also C52.2, C53.2, U11.11 (SD), U11.13 (VSS), U11.2 (COM), U15.5 (EM), U15.8 (EM), U18.11 (SD), U18.13 (VSS), U18.2 (COM)
- net I_C: now also U14.4
- net MCU_GND: now also U12.2 (V-), U13.5 (GND2), U14.2 (V-), U15.2 (CA), U15.3 (CA), U19.2 (V-)
- net at R30.1: now also U11.1 (LO)
- net at C39.2, R33.1, R35.2: now also U14.1 (+)
- net at C49.1, R38.2, R43.1: now also U14.3 (-)
- net at R23.2, U9.7 (COL): now also U11.10 (HIN)
- net at R24.2, U9.6 (COL): now also U11.12 (LIN)
- net at C28.2, C29.2, C30.2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: now also U10.2 (A), U11.5 (VS)
- net at C30.1, C31.1, R20.2: now also D2.1 (K), U11.6 (VB); no longer D3.1 (K)
- net at R25.1: now also U11.7 (HO)
- net at C49.2, R43.2: now also U19.3 (-), U19.4
- net at C11.1, C12.1, R4.1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: now also U17.1 (K)
- net at C11.2, C12.2, C13.2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: now also U17.2 (A)
- net at R45.2: now also U15.4 (AN)
- net at R41.1: now also U18.7 (HO)
- net at C47.1, C48.1, R36.2: now also D3.1 (K), U18.6 (VB)
- net at C45.2, C46.2, C47.2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: now also U13.4 (GND1), U16.2 (A), U18.5 (VS)
- net at C32.2, R27.2: now also U12.3 (-), U12.4
- net at R21.1, R28.2: no longer C27.2
- net at R21.2, U7.3 (INN): now also C27.2
- net at C28.1, C29.1, R20.1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: now also U10.1 (K)
- net at R18.1, R28.3: no longer C27.1
- net at R18.2, U7.2 (INP): now also C27.1
- net at C45.1, C46.1, R36.1: now also U13.1 (VDD1), U16.1 (K)
- net at R34.2: now also C44.1, U13.2 (INP)
- net at R37.2: now also C44.2, U13.3 (INN)
- net at R38.1: now also U13.6 (OUTN)
- net at R35.1: now also U13.7 (OUTP)
- net at R37.1, R44.2: no longer C44.2
- net at R42.2: now also U15.1 (AN)
- net at R40.2: now also U15.6 (COL), U18.12 (LIN)
- net at R39.2: now also U15.7 (COL), U18.10 (HIN)
- net at R46.1: now also U18.1 (LO)
- net at R12.2, R5.1: no longer C10.2
- net at R5.2, U2.3 (INN): now also C10.2
- net at R34.1, R44.3: no longer C44.1
- net at R12.3, R2.1: no longer C10.1
- net at R2.2, U2.2 (INP): now also C10.1
- net at R31.2, R32.1: now also U12.1 (+)
- net at R47.2, R48.1: now also U19.1 (+)
Other:
- moved on the sheet: C10, R2, R5

Commit message: Almost done
Connections:
- net +3.3V: now also J5.5 (Pin_5); no longer J5.4 (Pin_4)
- net MCU_GND: now also J5.4 (Pin_4); no longer J5.5 (Pin_5)
- net at R19.2, U8.1 (+): now also C32.1, R27.1; no longer C22.2, R17.1
- net at R22.2, U8.3 (-): now also C22.2, R17.1; no longer C32.1, R27.1
- net at C49.1, R43.1: now also R35.2, U14.1 (+); no longer R38.2, U14.3 (-)
- net at R3.2, U3.1 (+): now also C15.1, R11.1; no longer C5.2, R1.1
- net at C39.2, R33.1: now also R38.2, U14.3 (-); no longer R35.2, U14.1 (+)
- net at R6.2, U3.3 (-): now also C5.2, R1.1; no longer C15.1, R11.1
Other:
- moved on the sheet: C22, C39, C5, R1, R17, R33

Commit message: Done
Parts:
- R12, R28, R44: symbol Device:R_Shunt -> Device:R
Connections:
- net PHASE_A: now also R12.2, R2.1; no longer R12.4
- net PHASE_B: now also R18.1, R28.2; no longer R28.4
- net PHASE_C: now also R34.1, R44.2; no longer R44.4
- net at C28.2, C29.2, C30.2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: now also R21.1
- net at C11.2, C12.2, C13.2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: now also R5.1
- net at R37.1: now also C45.2, C46.2, C47.2, C48.2, Q5.3 (S), Q6.2 (D), R44.1, U13.4 (GND1), U16.2 (A), U18.5 (VS); no longer R44.2
Changed lines of the file:
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@@
 	)
 	(junction
+		(at 224.79 111.76)
+		(diameter 0)
+		(color 0 0 0 0)
+	)
+	(junction
+		(at 217.17 227.33)
+		(diameter 0)
+		(color 0 0 0 0)
+	)
+	(junction
 		(at 191.77 331.47)
 		(diameter 0)
@@
 	)
 	(junction
+		(at 217.17 342.9)
+		(diameter 0)
+		(color 0 0 0 0)
+	)
+	(junction
 		(at 127 88.9)
 		(diameter 0)
@@
 	)
 	(junction
+		(at 224.79 342.9)
+		(diameter 0)
+		(color 0 0 0 0)
+	)
+	(junction
 		(at 495.3 66.04)
 		(diameter 0)
@@
 	)
 	(junction
+		(at 217.17 111.76)
+		(diameter 0)
+		(color 0 0 0 0)
+	)
+	(junction
 		(at 279.4 256.54)
 		(diameter 0)
@@
 	)
 	(junction
+		(at 224.79 227.33)
+		(diameter 0)
+		(color 0 0 0 0)
+	)
+	(junction
 		(at 148.59 229.87)
 		(diameter 0)
@@
 	(wire
 		(pts
-			(xy 224.79 223.52) (xy 224.79 205.74)
+			(xy 74.93 81.28) (xy 95.25 81.28)
 		)
 		(stroke
@@
 	(wire
 		(pts
-			(xy 74.93 81.28) (xy 95.25 81.28)
+			(xy 323.85 71.12) (xy 330.2 71.12)
 		)
 		(stroke
@@
 	(wire
 		(pts
-			(xy 323.85 71.12) (xy 330.2 71.12)
+			(xy 90.17 232.41) (xy 91.44 232.41)
 		)
 		(stroke
@@
 	(wire
 		(pts
-			(xy 90.17 232.41) (xy 91.44 232.41)
+			(xy 128.27 334.01) (xy 128.27 332.74)
 		)
 		(stroke
@@
 	(wire
 		(pts
-			(xy 128.27 334.01) (xy 128.27 332.74)
+			(xy 287.02 227.33) (xy 287.02 229.87)
 		)
 		(stroke
@@
 	(wire
 		(pts
-			(xy 287.02 227.33) (xy 287.02 229.87)
+			(xy 217.17 213.36) (xy 217.17 227.33)
 		)
 		(stroke
@@
 	(wire
 		(pts
+			(xy 224.79 227.33) (xy 233.68 227.33)
+		)
+		(stroke
+			(width 0)
+			(type default)
+		)
+	)
+	(wire
+		(pts
 			(xy 115.57 81.28) (xy 115.57 96.52)
 		)
@@
 	(wire
 		(pts
-			(xy 224.79 107.95) (xy 224.79 90.17)
+			(xy 224.79 90.17) (xy 224.79 111.76)
 		)
 		(stroke
@@
 	(wire
 		(pts
-			(xy 224.79 339.09) (xy 224.79 321.31)
-		)
-		(stroke
-			(width 0)
-			(type default)
-		)
-	)
-	(wire
-		(pts
 			(xy 107.95 342.9) (xy 102.87 342.9)
 		)
@@
 	(wire
 		(pts
-			(xy 227.33 111.76) (xy 233.68 111.76)
-		)
-		(stroke
-			(width 0)
-			(type default)
-		)
-	)
-	(wire
-		(pts
 			(xy 127 320.04) (xy 142.24 320.04)
 		)
@@
 	(wire
 		(pts
-			(xy 219.71 223.52) (xy 219.71 213.36)
-		)
-		(stroke
-			(width 0)
-			(type default)
-		)
-	)
-	(wire
-		(pts
-			(xy 219.71 213.36) (xy 226.06 213.36)
+			(xy 217.17 213.36) (xy 226.06 213.36)
 		)
 		(stroke
@@
 	(wire
 		(pts
-			(xy 219.71 97.79) (xy 226.06 97.79)
+			(xy 217.17 97.79) (xy 226.06 97.79)
 		)
 		(stroke
@@
 	(wire
 		(pts
-			(xy 219.71 107.95) (xy 219.71 97.79)
+			(xy 217.17 97.79) (xy 217.17 111.76)
 		)
 		(stroke
@@
 	(wire
 		(pts
-			(xy 227.33 342.9) (xy 233.68 342.9)
-		)
-		(stroke
-			(width 0)
-			(type default)
-		)
-	)
-	(wire
-		(pts
 			(xy 134.62 227.33) (xy 175.26 227.33)
 		)
@@
 	(wire
 		(pts
-			(xy 219.71 339.09) (xy 219.71 328.93)
+			(xy 217.17 328.93) (xy 217.17 342.9)
 		)
 		(stroke
@@
 	(wire
 		(pts
+			(xy 224.79 111.76) (xy 233.68 111.76)
+		)
+		(stroke
+			(width 0)
+			(type default)
+		)
+	)
+	(wire
+		(pts
 			(xy 175.26 342.9) (xy 191.77 342.9)
 		)
@@
 	(wire
 		(pts
+			(xy 224.79 321.31) (xy 224.79 342.9)
+		)
+		(stroke
+			(width 0)
+			(type default)
+		)
+	)
+	(wire
+		(pts
 			(xy 148.59 110.49) (xy 148.59 114.3)
 		)
@@
 	(wire
 		(pts
+			(xy 224.79 205.74) (xy 224.79 227.33)
+		)
+		(stroke
+			(width 0)
+			(type default)
+		)
+	)
+	(wire
+		(pts
 			(xy 248.92 196.85) (xy 248.92 203.2)
 		)
@@
 	(wire
 		(pts
-			(xy 219.71 328.93) (xy 226.06 328.93)
+			(xy 217.17 328.93) (xy 226.06 328.93)
 		)
 		(stroke
@@
 	(wire
 		(pts
+			(xy 224.79 342.9) (xy 233.68 342.9)
+		)
+		(stroke
+			(width 0)
+			(type default)
+		)
+	)
+	(wire
+		(pts
 			(xy 251.46 68.58) (xy 262.89 68.58)
 		)
@@
 	(wire
 		(pts
-			(xy 227.33 227.33) (xy 233.68 227.33)
-		)
-		(stroke
-			(width 0)
-			(type default)
-		)
-	)
-	(wire
-		(pts
 			(xy 128.27 342.9) (xy 123.19 342.9)
 		)
@@
 	)
 	(symbol
-		(lib_id "Device:R_Shunt")
-		(at 222.25 111.76 90)
+		(lib_id "Device:R")
+		(at 220.98 111.76 90)
 		(unit 1)
 		(exclude_from_sim no)
@@
 		(on_board yes)
 		(dnp no)
-		(fields_autoplaced yes)
 		(property "Reference" "R12"
-			(at 222.25 115.57 90)
+			(at 223.52 118.11 90)
 			(effects
 				(font
@@
 		)
 		(property "Value" "R_Shunt"
-			(at 222.25 118.11 90)
+			(at 220.98 115.57 90)
 			(effects
 				(font
@@
 		)
 		(property "Footprint" "Custom_footprints:BVT-I-R003"
-			(at 222.25 113.538 90)
+			(at 220.98 113.538 90)
 			(effects
 				(font
@@
 		)
 		(property "Datasheet" "~"
-			(at 222.25 111.76 0)
+			(at 220.98 111.76 0)
 			(effects
 				(font
@@
 			)
 		)
-		(property "Description" "Shunt resistor"
-			(at 222.25 111.76 0)
+		(property "Description" "Resistor"
+			(at 220.98 111.76 0)
 			(effects
 				(font
@@
 			)
 		)
-		(pin "4"
-		)
 		(pin "1"
 		)
 		(pin "2"
 		)
-		(pin "3"
-		)
 		(instances
 			(project ""
@@
 	)
 	(symbol
-		(lib_id "Device:R_Shunt")
-		(at 222.25 342.9 90)
+		(lib_id "Device:R")
+		(at 220.98 342.9 90)
 		(unit 1)
 		(exclude_from_sim no)
@@
 		(fields_autoplaced yes)
 		(property "Reference" "R44"
-			(at 222.25 346.71 90)
+			(at 220.98 336.55 90)
 			(effects
 				(font
@@
 		)
 		(property "Value" "R_Shunt"
-			(at 222.25 349.25 90)
+			(at 220.98 339.09 90)
 			(effects
 				(font
@@
 		)
 		(property "Footprint" "Custom_footprints:BVT-I-R003"
-			(at 222.25 344.678 90)
+			(at 220.98 344.678 90)
 			(effects
 				(font
@@
 		)
 		(property "Datasheet" "~"
-			(at 222.25 342.9 0)
+			(at 220.98 342.9 0)
 			(effects
 				(font
@@
 			)
 		)
-		(property "Description" "Shunt resistor"
-			(at 222.25 342.9 0)
+		(property "Description" "Resistor"
+			(at 220.98 342.9 0)
 			(effects
 				(font
@@
 			)
 		)
-		(pin "4"
-		)
 		(pin "1"
 		)
 		(pin "2"
 		)
-		(pin "3"
-		)
 		(instances
 			(project "motor_driver"
@@
 	)
 	(symbol
-		(lib_id "Device:R_Shunt")
-		(at 222.25 227.33 90)
+		(lib_id "Device:R")
+		(at 220.98 227.33 90)
 		(unit 1)
 		(exclude_from_sim no)
@@
 		(fields_autoplaced yes)
 		(property "Reference" "R28"
-			(at 222.25 231.14 90)
+			(at 220.98 220.98 90)
 			(effects
 				(font
@@
 		)
 		(property "Value" "R_Shunt"
-			(at 222.25 233.68 90)
+			(at 220.98 223.52 90)
 			(effects
 				(font
@@
 		)
 		(property "Footprint" "Custom_footprints:BVT-I-R003_Reverse"
-			(at 222.25 229.108 90)
+			(at 220.98 229.108 90)
 			(effects
 				(font
@@
 		)
 		(property "Datasheet" "~"
-			(at 222.25 227.33 0)
+			(at 220.98 227.33 0)
 			(effects
 				(font
@@
 			)
 		)
-		(property "Description" "Shunt resistor"
-			(at 222.25 227.33 0)
+		(property "Description" "Resistor"
+			(at 220.98 227.33 0)
 			(effects
 				(font
@@
 			)
 		)
-		(pin "4"
-		)
-		(pin "1"
-		)
 		(pin "2"
 		)
-		(pin "3"
+		(pin "1"
 		)
 		(instances

Commit message: Add 3d models
Parts:
- J1: footprint TerminalBlock_MetzConnect:TerminalBlock_MetzConnect_Type067_RT01902HDWC_1x02_P10.00mm_Horizontal -> Custom_footprints:TerminalBlock_MetzConnect_Type067_RT01902HDWC_1x02_P10.00mm_Horizontal
- J2: footprint TerminalBlock:TerminalBlock_MaiXu_MX126-5.0-02P_1x02_P5.00mm -> Custom_footprints:TerminalBlock_MaiXu_MX126-5.0-02P_1x02_P5.00mm
- J3: footprint TerminalBlock_MetzConnect:TerminalBlock_MetzConnect_Type067_RT01903HDWC_1x03_P10.00mm_Horizontal -> Custom_footprints:TerminalBlock_MetzConnect_Type067_RT01903HDWC_1x03_P10.00mm_Horizontal
- U13, U2, U7: footprint Package_SO:SOIC-8_7.5x5.85mm_P1.27mm -> Custom_footprints:SOIC-8_7.5x5.85mm_P1.27mm
Changed lines of the file:
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@@
 			)
 		)
-		(property "Footprint" "Package_SO:SOIC-8_7.5x5.85mm_P1.27mm"
+		(property "Footprint" "Custom_footprints:SOIC-8_7.5x5.85mm_P1.27mm"
 			(at 251.46 210.82 0)
 			(effects
@@
 			)
 		)
-		(property "Footprint" "TerminalBlock_MetzConnect:TerminalBlock_MetzConnect_Type067_RT01902HDWC_1x02_P10.00mm_Horizontal"
+		(property "Footprint" "Custom_footprints:TerminalBlock_MetzConnect_Type067_RT01902HDWC_1x02_P10.00mm_Horizontal"
 			(at 403.86 77.47 0)
 			(effects
@@
 			)
 		)
-		(property "Footprint" "TerminalBlock_MetzConnect:TerminalBlock_MetzConnect_Type067_RT01903HDWC_1x03_P10.00mm_Horizontal"
+		(property "Footprint" "Custom_footprints:TerminalBlock_MetzConnect_Type067_RT01903HDWC_1x03_P10.00mm_Horizontal"
 			(at 504.19 110.49 0)
 			(effects
@@
 			)
 		)
-		(property "Footprint" "Package_SO:SOIC-8_7.5x5.85mm_P1.27mm"
+		(property "Footprint" "Custom_footprints:SOIC-8_7.5x5.85mm_P1.27mm"
 			(at 251.46 326.39 0)
 			(effects
@@
 			)
 		)
-		(property "Footprint" "TerminalBlock:TerminalBlock_MaiXu_MX126-5.0-02P_1x02_P5.00mm"
+		(property "Footprint" "Custom_footprints:TerminalBlock_MaiXu_MX126-5.0-02P_1x02_P5.00mm"
 			(at 445.77 77.47 0)
 			(effects
@@
 			)
 		)
-		(property "Footprint" "Package_SO:SOIC-8_7.5x5.85mm_P1.27mm"
+		(property "Footprint" "Custom_footprints:SOIC-8_7.5x5.85mm_P1.27mm"
 			(at 251.46 95.25 0)
 			(effects
